File: hardware/EAGLE/projects/DualMotorShield-v3.0/MotorShield.sch (EAGLE design)
At the start: 82 parts, among them IC2_1_CONN INTEL_BRD, U1 TSR_1-2450

Commit message: progress on DualModorShieldOnRaspberryHat
Parts:
- removed C10, C14, C15, C9, W_C4, W_C5: 0.22uF, SparkFun-Capacitors:0.22UF-0603-25V-10%
- removed C11, C13, C6, C8, W_C1, W_C3: 0.1uF, SparkFun-Capacitors:0.1UF-0603-25V-5%
- removed C12, C7, W_C2: 1nF, SparkFun-Capacitors:1.0NF/1000PF-0603-50V-10%
- removed H-BRIDGE2: PWM, SparkFun-Connectors:CONN_031X03_NO_SILK
- removed R10, R5, R6, R9, W_R3, W_R4: 10k, SparkFun-Resistors:10KOHM-0603-1/10W-1%
- removed R11, R7, W_R2: 47k, SparkFun-Resistors:47KOHM-0603-1/10W-1%
- removed R12, R8, W_R1: 4.7k, SparkFun-Resistors:4.7KOHM-0603-1/10W-1%
- removed SPI_CONN1: ENCODER, SparkFun-Connectors:CONN_06SMD-1MM
- removed U$1, U$2, U$3: (no value), ITX007T:IFX007TZZZZ
- removed U$10: TEENSY_3.1-3.2_ALL_PINS&PADS, Teensy_3_and_LC_Series_Boards_v1.4:TEENSY_3.1-3.2_ALL_PINS&PADS
- added H-BRIDGE0: BLDC0-PWM, SparkFun-Connectors:CONN_031X03_NO_SILK
- added SPI_CONN0: ENCODER0, SparkFun-Connectors:CONN_06SMD-1MM
- added U0_BRIDGE, V0_BRIDGE, W0_BRIDGE: (no value), ITX007T:IFX007TZZZZ
- added U0_C1, U0_C3, V0_C1, V0_C3, W0_C1, W0_C3: 0.1uF, SparkFun-Capacitors:0.1UF-0603-25V-5%
- added U0_C2, V0_C2, W0_C2: 1nF, SparkFun-Capacitors:1.0NF/1000PF-0603-50V-10%
- added U0_C4, U0_C5, V0_C4, V0_C5, W0_C4, W0_C5: 0.22uF, SparkFun-Capacitors:0.22UF-0603-25V-10%
- added U0_R1, V0_R1, W0_R1: 4.7k, SparkFun-Resistors:4.7KOHM-0603-1/10W-1%
- added U0_R2, V0_R2, W0_R2: 47k, SparkFun-Resistors:47KOHM-0603-1/10W-1%
- added U0_R3, U0_R4, V0_R3, V0_R4, W0_R3, W0_R4: 10k, SparkFun-Resistors:10KOHM-0603-1/10W-1%
- added X1: RASPI_BOARD_B+_H, raspberrypi_bastelstube_v13:RASPI_BOARD_B+_H
- H-BRIDGE1: value PWM -> BLDC1-PWM
- SPI_CONN2: value ENCODER -> ENCODER1
Connections:
- net U2 renamed PWN_U1
- net V2 renamed PWM_V1
- net W2 renamed PWM_W1
- removed net CS1: SPI_CONN1.5, U$10.9/RX2/PWM
- removed net CS2: SPI_CONN2.5, U$10.15/A1/T
- removed net INH_V: R9.2, U$10.3/CAN-TX/PWM
- removed net INH_W: U$10.33/T, W_R3.2
- removed net IN_U: H-BRIDGE1.3, R6.2
- removed net IN_U2_EX: U$10.21/A7/PWM
- removed net IN_U_EX: U$10.5/PWM
- removed net IN_V: H-BRIDGE1.2, R10.2
- removed net IN_V2_EX: U$10.22/A8/T/PWM
- removed net IN_V_EX: U$10.6/PWM
- removed net IN_W: H-BRIDGE1.1, W_R4.2
- removed net IN_W2_EX: U$10.23/A9/T/PWM
- removed net IN_W_EX: U$10.10/TX2/PWM
- removed net IS_U: C6.1, R8.2, U$1.IS, U$10.26/A15
- removed net IS_V: C11.1, R12.2, U$10.27/A16, U$3.IS
- removed net IS_W: U$10.28/A17, U$2.IS, W_C1.1, W_R1.2
- removed net MOSI: SPI_CONN1.2, SPI_CONN2.2, U$10.11/MOSI
- removed net SCK: SPI_CONN1.4, SPI_CONN2.4, U$10.13/SCK/LED
- removed net U: C10.2, C9.2, U$1.OUT, U$4.V
- removed net V: C14.2, C15.2, U$3.OUT, U$4.U
- removed net VI: C13.1, C14.1, C16.+, C19.1, C20.1, C24.1, C25.1, C3.1, C4.1, C8.1, C9.1, U$1.VS, U$2.VS, U$3.VS, U$5.2, U$6.VS, U$7.VS, U$9.VS, U1.VI, W_C3.1, W_C4.1
- removed net W: U$2.OUT, U$4.W, W_C4.2, W_C5.2
- new net INH_U0: X1.GPIO24
- new net INH_V0: V0_R3.2, X1.GPIO23
- new net INH_W0: W0_R3.2, X1.GPIO22
- new net IN_U0: H-BRIDGE0.3, U0_R4.2, X1.GPIO27
- new net IN_V0: H-BRIDGE0.2, V0_R4.2, X1.GPIO18
- new net IN_W0: H-BRIDGE0.1, W0_R4.2, X1.GPIO17
- new net IS_U0: U0_BRIDGE.IS, U0_C1.1, U0_R1.2, X1.GPIO04
- new net IS_V0: V0_BRIDGE.IS, V0_C1.1, V0_R1.2, X1.GPIO05
- new net IS_W0: W0_BRIDGE.IS, W0_C1.1, W0_R1.2, X1.GPIO25
- new net PWM_U0: U$4.V, U0_BRIDGE.OUT, U0_C4.2, U0_C5.2
- new net PWM_V0: U$4.U, V0_BRIDGE.OUT, V0_C4.2, V0_C5.2
- new net PWM_W0: U$4.W, W0_BRIDGE.OUT, W0_C4.2, W0_C5.2
- new net SPI_CE0: SPI_CONN0.5, X1.SPI_CE0
- new net SPI_CE1: SPI_CONN2.5, X1.SPI_CE1
- new net SPI_MISO: SPI_CONN0.3, X1.SPI_MISO
- new net SPI_MOSI: SPI_CONN0.2, SPI_CONN2.2, X1.SPI_MOSI
- new net SPI_SCLK: SPI_CONN0.4, SPI_CONN2.4, X1.SPI_SCLK
- new net VIN_BATTERY: C16.+, C19.1, C20.1, C24.1, C25.1, C3.1, C4.1, U$5.2, U$6.VS, U$7.VS, U$9.VS, U0_BRIDGE.VS, U0_C3.1, U0_C4.1, U1.VI, V0_BRIDGE.VS, V0_C3.1, V0_C4.1, W0_BRIDGE.VS, W0_C3.1, W0_C4.1
- net 3.3V: now also SPI_CONN0.1; no longer SPI_CONN1.1, U$10.3.3V
- net GND: now also SPI_CONN0.6, U0_BRIDGE.GND, U0_C1.2, U0_C2.1, U0_C3.2, U0_C5.1, U0_R1.1, U0_R2.1, V0_BRIDGE.GND, V0_C1.2, V0_C2.1, V0_C3.2, V0_C5.1, V0_R1.1, V0_R2.1, W0_BRIDGE.GND, W0_C1.2, W0_C2.1, W0_C3.2, W0_C5.1, W0_R1.1, W0_R2.1, X1.GND; no longer C10.1, C11.2, C12.1, C13.2, C15.1, C6.2, C7.1, C8.2, R11.1, R12.1, R7.1, R8.1, SPI_CONN1.6, U$1.GND, U$10.GND, U$2.GND, U$3.GND, W_C1.2, W_C2.1, W_C3.2, W_C5.1, W_R1.1, W_R2.1
- net HALL_U: no longer U$10.20/A6/PWM
- net HALL_U2: no longer U$10.14/A0
- net HALL_V: no longer U$10.A10
- net HALL_V2: no longer U$10.16/A2/T
- net HALL_W: no longer U$10.A11
- net HALL_W2: no longer U$10.17/A3/T
- net INH_U: now also U0_R3.2; no longer R5.2, U$10.24
- net INH_U2: no longer U$10.2
- net INH_V2: no longer U$10.1/TX1/T
- net INH_W2: no longer U$10.0/RX1/T
- net IN_U2: now also H-BRIDGE1.3; no longer H-BRIDGE2.3
- net IN_V2: now also H-BRIDGE1.2; no longer H-BRIDGE2.2
- net IN_W2: now also H-BRIDGE1.1; no longer H-BRIDGE2.1
- net IS_U2: no longer U$10.31/A20
- net IS_V2: no longer U$10.A13
- net IS_W2: no longer U$10.A12
- net MISO: no longer SPI_CONN1.3, U$10.12/MISO
- net N$1: now also W0_BRIDGE.INH, W0_R3.1; no longer U$2.INH, W_R3.1
- net N$10: now also U0_BRIDGE.SR, U0_C2.2, U0_R2.2; no longer C7.2, R7.2, U$1.SR
- net N$11: now also U0_BRIDGE.INH, U0_R3.1; no longer R5.1, U$1.INH
- net N$14: now also U0_BRIDGE.IN, U0_R4.1; no longer R6.1, U$1.IN
- net N$18: now also V0_BRIDGE.INH, V0_R3.1; no longer R9.1, U$3.INH
- net N$2: now also V0_BRIDGE.SR, V0_C2.2, V0_R2.2; no longer C12.2, R11.2, U$3.SR
- net N$20: now also W0_BRIDGE.IN, W0_R4.1; no longer U$2.IN, W_R4.1
- net N$24: now also V0_BRIDGE.IN, V0_R4.1; no longer R10.1, U$3.IN
- net N$3: now also W0_BRIDGE.SR, W0_C2.2, W0_R2.2; no longer U$2.SR, W_C2.2, W_R2.2
- net SCL0: no longer U$10.19/A5/T/SCL0
- net SCL1: no longer U$10.29/A18/SCL1
- net SDA0: no longer U$10.18/A4/T/SDA0
- net SDA1: no longer U$10.30/A19/SDA1
- net S_PWM_1: no longer U$10.32/T/PWM
- net S_PWM_2: no longer U$10.25/T/PWM
- net VCC: no longer U$10.VIN
Other:
- moved on the sheet: C1, C17, C18, C19, C2, C20, C21, C22, C23, C24, C25, C26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

Commit message: Dualboard update
Parts:
- removed U$7, U$9: (no value), ITX007T:IFX007TZZZZ
- added V1_BRIDGE, W1_BRIDGE: (no value), ITX007T:IFX007TZZZZ
Connections:
- net GND: now also V1_BRIDGE.GND, W1_BRIDGE.GND; no longer U$7.GND, U$9.GND
- net IS_V2: now also V1_BRIDGE.IS; no longer U$7.IS
- net IS_W2: now also W1_BRIDGE.IS; no longer U$9.IS
- net N$26: now also V1_BRIDGE.INH; no longer U$7.INH
- net N$27: now also V1_BRIDGE.IN; no longer U$7.IN
- net N$29: now also V1_BRIDGE.SR; no longer U$7.SR
- net N$30: now also W1_BRIDGE.INH; no longer U$9.INH
- net N$31: now also W1_BRIDGE.IN; no longer U$9.IN
- net N$33: now also W1_BRIDGE.SR; no longer U$9.SR
- net PWM_V1: now also V1_BRIDGE.OUT; no longer U$7.OUT
- net PWM_W1: now also W1_BRIDGE.OUT; no longer U$9.OUT
- net VIN_BATTERY: now also V1_BRIDGE.VS, W1_BRIDGE.VS; no longer U$7.VS, U$9.VS
Other:
- moved on the sheet: C19, C20, C21, C22, C23, C24, C25, C26, R20, R21, R22, R23

Commit message: minor updates on DualMotorShield-v3.0
Parts:
- removed C1, C17, C22, C3: 0.1uF, SparkFun-Capacitors:0.1UF-0603-25V-5%
- removed C18, C2: 1nF, SparkFun-Capacitors:1.0NF/1000PF-0603-50V-10%
- removed C20, C25, C4, C5: 0.22uF, SparkFun-Capacitors:0.22UF-0603-25V-10%
- removed H-BRIDGE0: BLDC0-PWM, SparkFun-Connectors:CONN_031X03_NO_SILK
- removed H-BRIDGE1: BLDC1-PWM, SparkFun-Connectors:CONN_031X03_NO_SILK
- removed R13, R16, R17, R20, R21, R4: 10k, SparkFun-Resistors:10KOHM-0603-1/10W-1%
- removed R14, R18: 47k, SparkFun-Resistors:47KOHM-0603-1/10W-1%
- removed R15, R19: 4.7k, SparkFun-Resistors:4.7KOHM-0603-1/10W-1%
- removed U$6: (no value), ITX007T:IFX007TZZZZ
- added U1_BRIDGE: (no value), ITX007T:IFX007TZZZZ
- added U1_C1, U1_C3, V1_C1, W1_C1: 0.1uF, SparkFun-Capacitors:0.1UF-0603-25V-5%
- added U1_C4, U1_C5, V1_C4, W1_C4: 0.22uF, SparkFun-Capacitors:0.22UF-0603-25V-10%
- added U1_D2, V1_C2: 1nF, SparkFun-Capacitors:1.0NF/1000PF-0603-50V-10%
- added U1_R1, V1_R1: 4.7k, SparkFun-Resistors:4.7KOHM-0603-1/10W-1%
- added U1_R2, V1_R2: 47k, SparkFun-Resistors:47KOHM-0603-1/10W-1%
- added U1_R3, U1_R4, V1_R3, V1_R4, W1_R3, W1_R4: 10k, SparkFun-Resistors:10KOHM-0603-1/10W-1%
- renumbered C19 to V1_C3, C21 to V1_C5, C23 to W1_C2, C24 to W1_C3, C26 to W1_C5, R22 to W1_R2, R23 to W1_R1
Connections:
- net HALL_U renamed HALL_U0
- net HALL_V renamed HALL_V0
- net HALL_W renamed HALL_W0
- removed net INH_U2: R4.2
- removed net INH_V2: R16.2
- removed net INH_W2: R20.2
- removed net IN_U2: H-BRIDGE1.3, R13.2
- removed net IN_V2: H-BRIDGE1.2, R17.2
- removed net IN_W2: H-BRIDGE1.1, R21.2
- removed net IS_U2: C1.1, R15.2, U$6.IS
- removed net IS_V2: C17.1, R19.2, V1_BRIDGE.IS
- removed net IS_W2: C22.1, W1_BRIDGE.IS, W1_R1.2
- new net INH_U1: U1_R3.2, X1.GPIO26
- new net INH_V1: V1_R3.2, X1.GPIO16
- new net INH_W1: W1_R3.2, X1.GPIO19
- new net IN_U1: U1_R4.2, X1.GPIO13
- new net IN_V1: V1_R4.2, X1.GPIO12
- new net IN_W1: W1_R4.2, X1.GPIO06
- new net IS_U1: U1_BRIDGE.IS, U1_C1.1, U1_R1.2
- new net IS_V1: V1_BRIDGE.IS, V1_C1.1, V1_R1.2, X1.GPIO21
- new net IS_W1: W1_BRIDGE.IS, W1_C1.1, W1_R1.2, X1.GPIO20
- new net IW_U1: X1.RXD
- net 3.3V: now also X1.3V3
- net GND: now also U1_BRIDGE.GND, U1_C1.2, U1_C3.2, U1_C5.1, U1_D2.1, U1_R1.1, U1_R2.1, V1_C1.2, V1_C2.1, V1_R1.1, V1_R2.1, W1_C1.2; no longer C1.2, C17.2, C18.1, C2.1, C22.2, C3.2, C5.1, R14.1, R15.1, R18.1, R19.1, U$6.GND
- net IN_U0: no longer H-BRIDGE0.3
- net IN_V0: no longer H-BRIDGE0.2
- net IN_W0: no longer H-BRIDGE0.1
- net N$17: now also U1_BRIDGE.INH, U1_R3.1; no longer R4.1, U$6.INH
- net N$19: now also U1_BRIDGE.IN, U1_R4.1; no longer R13.1, U$6.IN
- net N$23: now also U1_BRIDGE.SR, U1_D2.2, U1_R2.2; no longer C2.2, R14.2, U$6.SR
- net N$26: now also V1_R3.1; no longer R16.1
- net N$27: now also V1_R4.1; no longer R17.1
- net N$29: now also V1_C2.2, V1_R2.2; no longer C18.2, R18.2
- net N$30: now also W1_R3.1; no longer R20.1
- net N$31: now also W1_R4.1; no longer R21.1
- net PWM_V1: now also V1_C4.2; no longer C20.2
- net PWM_W1: now also W1_C4.2; no longer C25.2
- net PWN_U1: now also U1_BRIDGE.OUT, U1_C4.2, U1_C5.2; no longer C4.2, C5.2, U$6.OUT
- net SCL0: now also X1.SCL
- net SCL1: now also X1.ID_SC
- net SDA0: now also X1.SDA
- net SDA1: now also X1.ID_SD
- net VCC: now also X1.5V0
- net VIN_BATTERY: now also U1_BRIDGE.VS, U1_C3.1, U1_C4.1, V1_C4.1, W1_C4.1; no longer C20.1, C25.1, C3.1, C4.1, U$6.VS
Other:
- moved on the sheet: C16, HALL, HALL1, I2C_2_CONN, IC2_1_CONN, R1, R2, R24, R25, R26, R3, SERVO_1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

Commit message: DualShield update
Parts:
- removed SPI_CONN0: ENCODER0, SparkFun-Connectors:CONN_06SMD-1MM
- removed U0_BRIDGE, U1_BRIDGE, V0_BRIDGE, V1_BRIDGE, W0_BRIDGE, W1_BRIDGE: (no value), ITX007T:IFX007TZZZZ
- removed U0_C1, U0_C3, U1_C1, U1_C3, V0_C1, V0_C3, V1_C1, V1_C3, W0_C1, W0_C3, W1_C1, W1_C3: 0.1uF, SparkFun-Capacitors:0.1UF-0603-25V-5%
- removed U0_C2, U1_D2, V0_C2, V1_C2, W0_C2, W1_C2: 1nF, SparkFun-Capacitors:1.0NF/1000PF-0603-50V-10%
- removed U0_C4, U0_C5, U1_C4, U1_C5, V0_C4, V0_C5, V1_C4, V1_C5, W0_C4, W0_C5, W1_C4, W1_C5: 0.22uF, SparkFun-Capacitors:0.22UF-0603-25V-10%
- removed U0_R1, U1_R1, V0_R1, V1_R1, W0_R1, W1_R1: 4.7k, SparkFun-Resistors:4.7KOHM-0603-1/10W-1%
- removed U0_R2, U1_R2, V0_R2, V1_R2, W0_R2, W1_R2: 47k, SparkFun-Resistors:47KOHM-0603-1/10W-1%
- removed U0_R3, U0_R4, U1_R3, U1_R4, V0_R3, V0_R4, V1_R3, V1_R4, W0_R3, W0_R4, W1_R3, W1_R4: 10k, SparkFun-Resistors:10KOHM-0603-1/10W-1%
- removed X1: RASPI_BOARD_B+_H, raspberrypi_bastelstube_v13:RASPI_BOARD_B+_H
- added C1, C11, C13, C17, C19, C22, C24, C3, C6, C8, W_C1, W_C3: 0.1uF, SparkFun-Capacitors:0.1UF-0603-25V-5%
- added C10, C14, C15, C20, C21, C25, C26, C4, C5, C9, W_C4, W_C5: 0.22uF, SparkFun-Capacitors:0.22UF-0603-25V-10%
- added C12, C18, C2, C23, C7, W_C2: 1nF, SparkFun-Capacitors:1.0NF/1000PF-0603-50V-10%
- added H-BRIDGE1, H-BRIDGE2: PWM, SparkFun-Connectors:CONN_031X03_NO_SILK
- added R10, R13, R16, R17, R20, R21, R4, R5, R6, R9, W_R3, W_R4: 10k, SparkFun-Resistors:10KOHM-0603-1/10W-1%
- added R11, R14, R18, R22, R7, W_R2: 47k, SparkFun-Resistors:47KOHM-0603-1/10W-1%
- added R12, R15, R19, R23, R8, W_R1: 4.7k, SparkFun-Resistors:4.7KOHM-0603-1/10W-1%
- added SPI_CONN1: ENCODER, SparkFun-Connectors:CONN_06SMD-1MM
- added U$1, U$2, U$3, U$6, U$7, U$9: (no value), ITX007T:IFX007TZZZZ
- added U$10: TEENSY_3.1-3.2_ALL_PINS&PADS, Teensy_3_and_LC_Series_Boards_v1.4:TEENSY_3.1-3.2_ALL_PINS&PADS
- SPI_CONN2: value ENCODER1 -> ENCODER
Connections:
- removed net HALL_U0: HALL.2, R2.1
- removed net HALL_V0: HALL.3, R3.1
- removed net HALL_W0: HALL.4, R1.1
- removed net INH_U0: X1.GPIO24
- removed net INH_U1: U1_R3.2, X1.GPIO26
- removed net INH_V0: V0_R3.2, X1.GPIO23
- removed net INH_V1: V1_R3.2, X1.GPIO16
- removed net INH_W0: W0_R3.2, X1.GPIO22
- removed net INH_W1: W1_R3.2, X1.GPIO19
- removed net IN_U0: U0_R4.2, X1.GPIO27
- removed net IN_U1: U1_R4.2, X1.GPIO13
- removed net IN_V0: V0_R4.2, X1.GPIO18
- removed net IN_V1: V1_R4.2, X1.GPIO12
- removed net IN_W0: W0_R4.2, X1.GPIO17
- removed net IN_W1: W1_R4.2, X1.GPIO06
- removed net IS_U0: U0_BRIDGE.IS, U0_C1.1, U0_R1.2, X1.GPIO04
- removed net IS_U1: U1_BRIDGE.IS, U1_C1.1, U1_R1.2
- removed net IS_V0: V0_BRIDGE.IS, V0_C1.1, V0_R1.2, X1.GPIO05
- removed net IS_V1: V1_BRIDGE.IS, V1_C1.1, V1_R1.2, X1.GPIO21
- removed net IS_W0: W0_BRIDGE.IS, W0_C1.1, W0_R1.2, X1.GPIO25
- removed net IS_W1: W1_BRIDGE.IS, W1_C1.1, W1_R1.2, X1.GPIO20
- removed net IW_U1: X1.RXD
- removed net PWM_U0: U$4.V, U0_BRIDGE.OUT, U0_C4.2, U0_C5.2
- removed net PWM_V0: U$4.U, V0_BRIDGE.OUT, V0_C4.2, V0_C5.2
- removed net PWM_V1: U$8.U, V1_BRIDGE.OUT, V1_C4.2, V1_C5.2
- removed net PWM_W0: U$4.W, W0_BRIDGE.OUT, W0_C4.2, W0_C5.2
- removed net PWM_W1: U$8.V, W1_BRIDGE.OUT, W1_C4.2, W1_C5.2
- removed net PWN_U1: U$8.W, U1_BRIDGE.OUT, U1_C4.2, U1_C5.2
- removed net SPI_CE0: SPI_CONN0.5, X1.SPI_CE0
- removed net SPI_CE1: SPI_CONN2.5, X1.SPI_CE1
- removed net SPI_MISO: SPI_CONN0.3, X1.SPI_MISO
- removed net SPI_MOSI: SPI_CONN0.2, SPI_CONN2.2, X1.SPI_MOSI
- removed net SPI_SCLK: SPI_CONN0.4, SPI_CONN2.4, X1.SPI_SCLK
- removed net VIN_BATTERY: C16.+, U$5.2, U0_BRIDGE.VS, U0_C3.1, U0_C4.1, U1.VI, U1_BRIDGE.VS, U1_C3.1, U1_C4.1, V0_BRIDGE.VS, V0_C3.1, V0_C4.1, V1_BRIDGE.VS, V1_C3.1, V1_C4.1, W0_BRIDGE.VS, W0_C3.1, W0_C4.1, W1_BRIDGE.VS, W1_C3.1, W1_C4.1
- new net CS1: SPI_CONN1.5, U$10.9/RX2/PWM
- new net CS2: SPI_CONN2.5, U$10.15/A1/T
- new net HALL_U: HALL.2, R2.1, U$10.20/A6/PWM
- new net HALL_V: HALL.3, R3.1, U$10.A10
- new net HALL_W: HALL.4, R1.1, U$10.A11
- new net INH_U2: R4.2, U$10.2
- new net INH_V: R9.2, U$10.3/CAN-TX/PWM
- new net INH_V2: R16.2, U$10.1/TX1/T
- new net INH_W: U$10.33/T, W_R3.2
- new net INH_W2: R20.2, U$10.0/RX1/T
- new net IN_U: H-BRIDGE1.3, R6.2
- new net IN_U2: H-BRIDGE2.3, R13.2
- new net IN_U2_EX: U$10.21/A7/PWM
- new net IN_U_EX: U$10.5/PWM
- new net IN_V: H-BRIDGE1.2, R10.2
- new net IN_V2: H-BRIDGE2.2, R17.2
- new net IN_V2_EX: U$10.22/A8/T/PWM
- new net IN_V_EX: U$10.6/PWM
- new net IN_W: H-BRIDGE1.1, W_R4.2
- new net IN_W2: H-BRIDGE2.1, R21.2
- new net IN_W2_EX: U$10.23/A9/T/PWM
- new net IN_W_EX: U$10.10/TX2/PWM
- new net IS_U: C6.1, R8.2, U$1.IS, U$10.26/A15
- new net IS_U2: C1.1, R15.2, U$10.31/A20, U$6.IS
- new net IS_V: C11.1, R12.2, U$10.27/A16, U$3.IS
- new net IS_V2: C17.1, R19.2, U$10.A13, U$7.IS
- new net IS_W: U$10.28/A17, U$2.IS, W_C1.1, W_R1.2
- new net IS_W2: C22.1, R23.2, U$10.A12, U$9.IS
- new net MOSI: SPI_CONN1.2, SPI_CONN2.2, U$10.11/MOSI
- new net SCK: SPI_CONN1.4, SPI_CONN2.4, U$10.13/SCK/LED
- new net U: C10.2, C9.2, U$1.OUT, U$4.V
- new net U2: C4.2, C5.2, U$6.OUT, U$8.W
- new net V: C14.2, C15.2, U$3.OUT, U$4.U
- new net V2: C20.2, C21.2, U$7.OUT, U$8.U
- new net VI: C13.1, C14.1, C16.+, C19.1, C20.1, C24.1, C25.1, C3.1, C4.1, C8.1, C9.1, U$1.VS, U$2.VS, U$3.VS, U$5.2, U$6.VS, U$7.VS, U$9.VS, U1.VI, W_C3.1, W_C4.1
- new net W: U$2.OUT, U$4.W, W_C4.2, W_C5.2
- new net W2: C25.2, C26.2, U$8.V, U$9.OUT
- net 3.3V: now also SPI_CONN1.1, U$10.3.3V; no longer SPI_CONN0.1, X1.3V3
- net GND: now also C1.2, C10.1, C11.2, C12.1, C13.2, C15.1, C17.2, C18.1, C19.2, C2.1, C21.1, C22.2, C23.1, C24.2, C26.1, C3.2, C5.1, C6.2, C7.1, C8.2, R11.1, R12.1, R14.1, R15.1, R18.1, R19.1, R22.1, R23.1, R7.1, R8.1, SPI_CONN1.6, U$1.GND, U$10.GND, U$2.GND, U$3.GND, U$6.GND, U$7.GND, U$9.GND, W_C1.2, W_C2.1, W_C3.2, W_C5.1, W_R1.1, W_R2.1; no longer SPI_CONN0.6, U0_BRIDGE.GND, U0_C1.2, U0_C2.1, U0_C3.2, U0_C5.1, U0_R1.1, U0_R2.1, U1_BRIDGE.GND, U1_C1.2, U1_C3.2, U1_C5.1, U1_D2.1, U1_R1.1, U1_R2.1, V0_BRIDGE.GND, V0_C1.2, V0_C2.1, V0_C3.2, V0_C5.1, V0_R1.1, V0_R2.1, V1_BRIDGE.GND, V1_C1.2, V1_C2.1, V1_C3.2, V1_C5.1, V1_R1.1, V1_R2.1, W0_BRIDGE.GND, W0_C1.2, W0_C2.1, W0_C3.2, W0_C5.1, W0_R1.1, W0_R2.1, W1_BRIDGE.GND, W1_C1.2, W1_C2.1, W1_C3.2, W1_C5.1, W1_R1.1, W1_R2.1, X1.GND
- net HALL_U2: now also U$10.14/A0
- net HALL_V2: now also U$10.16/A2/T
- net HALL_W2: now also U$10.17/A3/T
- net INH_U: now also R5.2, U$10.24; no longer U0_R3.2
- net MISO: now also SPI_CONN1.3, U$10.12/MISO
- net N$1: now also U$2.INH, W_R3.1; no longer W0_BRIDGE.INH, W0_R3.1
- net N$10: now also C7.2, R7.2, U$1.SR; no longer U0_BRIDGE.SR, U0_C2.2, U0_R2.2
- net N$11: now also R5.1, U$1.INH; no longer U0_BRIDGE.INH, U0_R3.1
- net N$14: now also R6.1, U$1.IN; no longer U0_BRIDGE.IN, U0_R4.1
- net N$17: now also R4.1, U$6.INH; no longer U1_BRIDGE.INH, U1_R3.1
- net N$18: now also R9.1, U$3.INH; no longer V0_BRIDGE.INH, V0_R3.1
- net N$19: now also R13.1, U$6.IN; no longer U1_BRIDGE.IN, U1_R4.1
- net N$2: now also C12.2, R11.2, U$3.SR; no longer V0_BRIDGE.SR, V0_C2.2, V0_R2.2
- net N$20: now also U$2.IN, W_R4.1; no longer W0_BRIDGE.IN, W0_R4.1
- net N$23: now also C2.2, R14.2, U$6.SR; no longer U1_BRIDGE.SR, U1_D2.2, U1_R2.2
- net N$24: now also R10.1, U$3.IN; no longer V0_BRIDGE.IN, V0_R4.1
- net N$26: now also R16.1, U$7.INH; no longer V1_BRIDGE.INH, V1_R3.1
- net N$27: now also R17.1, U$7.IN; no longer V1_BRIDGE.IN, V1_R4.1
- net N$29: now also C18.2, R18.2, U$7.SR; no longer V1_BRIDGE.SR, V1_C2.2, V1_R2.2
- net N$3: now also U$2.SR, W_C2.2, W_R2.2; no longer W0_BRIDGE.SR, W0_C2.2, W0_R2.2
- net N$30: now also R20.1, U$9.INH; no longer W1_BRIDGE.INH, W1_R3.1
- net N$31: now also R21.1, U$9.IN; no longer W1_BRIDGE.IN, W1_R4.1
- net N$33: now also C23.2, R22.2, U$9.SR; no longer W1_BRIDGE.SR, W1_C2.2, W1_R2.2
- net SCL0: now also U$10.19/A5/T/SCL0; no longer X1.SCL
- net SCL1: now also U$10.29/A18/SCL1; no longer X1.ID_SC
- net SDA0: now also U$10.18/A4/T/SDA0; no longer X1.SDA
- net SDA1: now also U$10.30/A19/SDA1; no longer X1.ID_SD
- net S_PWM_1: now also U$10.32/T/PWM
- net S_PWM_2: now also U$10.25/T/PWM
- net VCC: now also U$10.VIN; no longer X1.5V0
Other:
- moved on the sheet: C16, HALL, HALL1, I2C_2_CONN, IC2_1_CONN, R1, R2, R24, R25, R26, R3, SERVO_1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

Commit message: spi update
Parts:
- removed U$4, U$8: (no value), 5569-03:5569-003
- added MOTOR0, MOTOR1: PWM, SparkFun-Connectors:CONN_031X03_NO_SILK
Connections:
- net 3.3V: now also SPI_CONN1.5, SPI_CONN2.5; no longer SPI_CONN1.1, SPI_CONN2.1
- net CS1: now also SPI_CONN1.1; no longer SPI_CONN1.5
- net CS2: now also SPI_CONN2.1; no longer SPI_CONN2.5
- net MISO: now also SPI_CONN1.4, SPI_CONN2.4; no longer SPI_CONN1.3, SPI_CONN2.3
- net MOSI: now also SPI_CONN1.3, SPI_CONN2.3; no longer SPI_CONN1.2, SPI_CONN2.2
- net SCK: now also SPI_CONN1.2, SPI_CONN2.2; no longer SPI_CONN1.4, SPI_CONN2.4
- net U: now also MOTOR0.1; no longer U$4.V
- net U2: now also MOTOR1.1; no longer U$8.W
- net V: now also MOTOR0.2; no longer U$4.U
- net V2: now also MOTOR1.2; no longer U$8.U
- net W: now also MOTOR0.3; no longer U$4.W
- net W2: now also MOTOR1.3; no longer U$8.V
Other:
- moved on the sheet: HALL1, SPI_CONN2

Commit message: Component renamed
Parts:
- removed SPI_CONN2: ENCODER, SparkFun-Connectors:CONN_06SMD-1MM
- added SPI_CONN0: ENCODER0, SparkFun-Connectors:CONN_06SMD-1MM
- I2C_1_IMU: value IMU_SENS -> JP
- IC2_0_PC: value INTEL_BRD -> JP
- IN-PWM0, IN-PWM1, MOTOR0, MOTOR1: value PWM -> JP
- SERVO_0, SERVO_1: value (none) -> JP
- SPI_CONN1: value ENCODER -> ENCODER1
- renumbered C1 to U1-C1, C10 to U0-C3, C11 to V0-C1, C12 to V0-C2, C13 to V0-C4, C14 to V0-C5, C15 to V0-C3, C16 to C0, C17 to V1-C1, C18 to V1-C2, C19 to V1-C4, C2 to U1-C2, C20 to V1-C5, C21 to V1-C3, C22 to W1-C1, C23 to W1-C2, C24 to W1-C4, C25 to W1-C5, C26 to W1-C3, C3 to U1-C4, C4 to U1-C5, C5 to U1-C3, C6 to U0-C1, C7 to U0-C2, C8 to U0-C4, C9 to U0-C5, H-BRIDGE1 to IN-PWM0, H-BRIDGE2 to IN-PWM1, HALL to HALL0, I2C_2_CONN to I2C_1_IMU, IC2_1_CONN to IC2_0_PC, R1 to H0-R1, R10 to V0-R4, R11 to V0-R2, R12 to V0-R1, R13 to U1-R4, R14 to U1-R2, R15 to U1-R1, R16 to V1-R3, R17 to V1-R4, R18 to V1-R2, R19 to V1-R1, R2 to H0-R3, R20 to W1-R3, R21 to W1-R4, R22 to W1-R2, R23 to W1-R1, R24 to H1-R1, R25 to H1-R3, R26 to H1-R2, R3 to H0-R2, R4 to U1-R3, R5 to U0-R3, R6 to U0-R4, R7 to U0-R2, R8 to U0-R1, R9 to V0-R3, SERVO_2 to SERVO_0, U$1 to HB-U0, U$10 to IC0, U$2 to HB-W0, U$3 to HB-V0, U$6 to HB-U1, U$7 to HB-V1, U$9 to HB-W1, W_C1 to W0-C1, W_C2 to W0-C2, W_C3 to W0-C4, W_C4 to W0-C5, W_C5 to W0-C3, W_R1 to W0-R1, W_R2 to W0-R2, W_R3 to W0-R3, W_R4 to W0-R4
Connections:
- net HALL_U renamed HALL_U0
- net HALL_V renamed HALL_V0
- net HALL_W renamed HALL_W0
- net INH_U renamed INH_U0
- net INH_U2 renamed INH_U1
- net INH_V renamed INH_V0
- net INH_V2 renamed INH_V1
- net INH_W renamed INH_W0
- net INH_W2 renamed INH_W1
- net IN_U renamed IN_U0
- net IN_U2 renamed IN_U1
- net IN_V renamed IN_V0
- net IN_V2 renamed IN_V1
- net IN_W renamed IN_W0
- net IN_W2 renamed IN_W1
- net IS_U renamed IS_U0
- net IS_U2 renamed IS_U1
- net IS_V renamed IS_V0
- net IS_V2 renamed IS_V1
- net IS_W renamed IS_W0
- net IS_W2 renamed IS_W1
- net U renamed U0
- net U2 renamed U1
- net V renamed V0
- net V2 renamed V1
- net W renamed W0
- net W2 renamed W1
- net 3.3V: now also SPI_CONN0.5; no longer SPI_CONN2.5
- net CS1: now also SPI_CONN0.1; no longer SPI_CONN1.1
- net CS2: now also SPI_CONN1.1; no longer SPI_CONN2.1
- net GND: now also SPI_CONN0.6; no longer SPI_CONN2.6
- net MISO: now also SPI_CONN0.4; no longer SPI_CONN2.4
- net MOSI: now also SPI_CONN0.3; no longer SPI_CONN2.3
- net SCK: now also SPI_CONN0.2; no longer SPI_CONN2.2
Other:
- moved on the sheet: SPI_CONN1
