File: hardware/EAGLE/projects/PiHatTeensy32/PiHatTeensy32.brd (EAGLE design)
At the start: 100 x 80 mm, 11 parts, among them U1 TSR_1-2450, X1 RASPI_BOARD_B+_H

Commit message: schematic connection done, pins 16-17 should be wired to UART
Connections:
- new net N$4: U$1.3
- net HALL_U0: now also U$1.0
- net HALL_U1: now also U$1.1
- net HALL_V0: now also U$1.24
- net HALL_V1: now also U$1.2
- net HALL_W0: now also U$1.33
- net HALL_W1: now also U$1.4
- net I2C0_SCL: now also U$1.29
- net I2C0_SDA: now also U$1.30
- net IN_U0: now also U$1.23/A9
- net IN_U1: now also U$1.5
- net IN_V0: now also U$1.22/A8
- net IN_V1: now also U$1.6
- net IN_W0: now also U$1.21/A7
- net IN_W1: now also U$1.10
- net IS_U0: now also U$1.20/A6
- net IS_U1: now also U$1.26
- net IS_V0: now also U$1.19/A5
- net IS_V1: now also U$1.27
- net IS_W0: now also U$1.18/A4
- net IS_W1: now also U$1.28
- net SERVO_0: now also U$1.32
- net SERVO_1: now also U$1.25
- net SPI_CS0: now also U$1.15/A1
- net SPI_CS1: now also U$1.31
- net SPI_MISO: now also U$1.12
- net SPI_MOSI: now also U$1.11
- net SPI_SCLK: now also U$1.14/A0
Changed lines of the file:
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@@
 <?xml version="1.0" encoding="utf-8"?>
 <!DOCTYPE eagle SYSTEM "eagle.dtd">
-<eagle version="9.6.0">
+<eagle version="9.5.2">
 <drawing>
 <settings>
@@
 <signal name="IN_U0">
 <contactref element="MOTOR0_CONTROL" pad="4"/>
+<contactref element="U$1" pad="23/A9"/>
+<wire x1="25.4" y1="19.05" x2="8.89" y2="41.91" width="0" layer="19" extent="1-1"/>
 </signal>
 <signal name="IN_V0">
 <contactref element="MOTOR0_CONTROL" pad="5"/>
+<contactref element="U$1" pad="22/A8"/>
+<wire x1="25.4" y1="21.59" x2="8.89" y2="44.45" width="0" layer="19" extent="1-1"/>
 </signal>
 <signal name="IN_W0">
 <contactref element="MOTOR0_CONTROL" pad="6"/>
+<contactref element="U$1" pad="21/A7"/>
+<wire x1="25.4" y1="24.13" x2="8.89" y2="46.99" width="0" layer="19" extent="1-1"/>
 </signal>
 <signal name="INH_U0">
@@
 <signal name="IS_W0">
 <contactref element="MOTOR0_SENS" pad="6"/>
+<contactref element="U$1" pad="18/A4"/>
+<wire x1="8.89" y1="24.13" x2="25.4" y2="31.75" width="0" layer="19" extent="1-1"/>
 </signal>
 <signal name="IS_V0">
 <contactref element="MOTOR0_SENS" pad="5"/>
+<contactref element="U$1" pad="19/A5"/>
+<wire x1="8.89" y1="21.59" x2="25.4" y2="29.21" width="0" layer="19" extent="1-1"/>
 </signal>
 <signal name="IS_U0">
 <contactref element="MOTOR0_SENS" pad="4"/>
+<contactref element="U$1" pad="20/A6"/>
+<wire x1="8.89" y1="19.05" x2="25.4" y2="26.67" width="0" layer="19" extent="1-1"/>
 </signal>
 <signal name="VI">
@@
 <signal name="IN_U1">
 <contactref element="MOTOR1_CONTROL" pad="4"/>
+<contactref element="U$1" pad="5"/>
+<wire x1="40.64" y1="26.67" x2="57.15" y2="41.91" width="0" layer="19" extent="1-1"/>
 </signal>
 <signal name="IN_V1">
 <contactref element="MOTOR1_CONTROL" pad="5"/>
+<contactref element="U$1" pad="6"/>
+<wire x1="40.64" y1="29.21" x2="57.15" y2="44.45" width="0" layer="19" extent="1-1"/>
 </signal>
 <signal name="IN_W1">
 <contactref element="MOTOR1_CONTROL" pad="6"/>
+<contactref element="U$1" pad="10"/>
+<wire x1="40.64" y1="39.37" x2="57.15" y2="46.99" width="0" layer="19" extent="1-1"/>
 </signal>
 <signal name="INH_V1">
@@
 <signal name="IS_W1">
 <contactref element="MOTOR1_SENS" pad="6"/>
+<contactref element="U$1" pad="28"/>
+<wire x1="33.02" y1="41.91" x2="57.15" y2="24.13" width="0" layer="19" extent="1-1"/>
 </signal>
 <signal name="IS_V1">
 <contactref element="MOTOR1_SENS" pad="5"/>
+<contactref element="U$1" pad="27"/>
+<wire x1="33.02" y1="39.37" x2="57.15" y2="21.59" width="0" layer="19" extent="1-1"/>
 </signal>
 <signal name="IS_U1">
 <contactref element="MOTOR1_SENS" pad="4"/>
+<contactref element="U$1" pad="26"/>
+<wire x1="33.02" y1="36.83" x2="57.15" y2="19.05" width="0" layer="19" extent="1-1"/>
 </signal>
 <signal name="I2C1_SDA">
@@
 <signal name="I2C0_SDA">
 <contactref element="X1" pad="3"/>
+<contactref element="U$1" pad="30"/>
+<wire x1="11.428159375" y1="52.07074375" x2="30.48" y2="39.37" width="0" layer="19" extent="1-1"/>
 </signal>
 <signal name="I2C0_SCL">
 <contactref element="X1" pad="5"/>
+<contactref element="U$1" pad="29"/>
+<wire x1="13.968159375" y1="52.07074375" x2="30.48" y2="41.91" width="0" layer="19" extent="1-1"/>
 </signal>
 <signal name="SPI_SCLK">
 <contactref element="X1" pad="23"/>
+<contactref element="U$1" pad="14/A0"/>
+<wire x1="25.4" y1="41.91" x2="36.828159375" y2="52.07074375" width="0" layer="19" extent="1-1"/>
 </signal>
 <signal name="SPI_MOSI">
 <contactref element="X1" pad="19"/>
+<contactref element="U$1" pad="11"/>
+<wire x1="40.64" y1="41.91" x2="31.748159375" y2="52.07074375" width="0" layer="19" extent="1-1"/>
 </signal>
 <signal name="SPI_MISO">
 <contactref element="X1" pad="21"/>
+<contactref element="U$1" pad="12"/>
+<wire x1="40.64" y1="44.45" x2="34.288159375" y2="52.07074375" width="0" layer="19" extent="1-1"/>
 </signal>
 <signal name="SPI_CS1">
 <contactref element="X1" pad="26"/>
+<contactref element="U$1" pad="31"/>
+<wire x1="30.48" y1="36.83" x2="39.368159375" y2="54.61074375" width="0" layer="19" extent="1-1"/>
 </signal>
 <signal name="SPI_CS0">
 <contactref element="X1" pad="24"/>
+<contactref element="U$1" pad="15/A1"/>
+<wire x1="25.4" y1="39.37" x2="36.828159375" y2="54.61074375" width="0" layer="19" extent="1-1"/>
 </signal>
 <signal name="HALL_U0">
 <contactref element="MOTOR0_SENS" pad="1"/>
+<contactref element="U$1" pad="0"/>
+<wire x1="8.89" y1="11.43" x2="40.64" y2="13.97" width="0" layer="19" extent="1-1"/>
 </signal>
 <signal name="HALL_V0">
 <contactref element="MOTOR0_SENS" pad="2"/>
+<contactref element="U$1" pad="24"/>
+<wire x1="8.89" y1="13.97" x2="33.02" y2="31.75" width="0" layer="19" extent="1-1"/>
 </signal>
 <signal name="HALL_W0">
 <contactref element="MOTOR0_SENS" pad="3"/>
+<contactref element="U$1" pad="33"/>
+<wire x1="8.89" y1="16.51" x2="30.48" y2="31.75" width="0" layer="19" extent="1-1"/>
 </signal>
 <signal name="SERVO_0">
 <contactref element="SERVOS" pad="1"/>
+<contactref element="U$1" pad="32"/>
+<wire x1="11.43" y1="11.43" x2="30.48" y2="34.29" width="0" layer="19" extent="1-1"/>
 </signal>
 <signal name="HALL_U1">
 <contactref element="MOTOR1_SENS" pad="1"/>
+<contactref element="U$1" pad="1"/>
+<wire x1="40.64" y1="16.51" x2="57.15" y2="11.43" width="0" layer="19" extent="1-1"/>
 </signal>
 <signal name="HALL_V1">
 <contactref element="MOTOR1_SENS" pad="2"/>
+<contactref element="U$1" pad="2"/>
+<wire x1="40.64" y1="19.05" x2="57.15" y2="13.97" width="0" layer="19" extent="1-1"/>
 </signal>
 <signal name="HALL_W1">
 <contactref element="MOTOR1_SENS" pad="3"/>
+<contactref element="U$1" pad="4"/>
+<wire x1="40.64" y1="24.13" x2="57.15" y2="16.51" width="0" layer="19" extent="1-1"/>
 </signal>
 <signal name="SERVO_1">
 <contactref element="SERVOS" pad="2"/>
+<contactref element="U$1" pad="25"/>
+<wire x1="13.97" y1="11.43" x2="33.02" y2="34.29" width="0" layer="19" extent="1-1"/>
 </signal>
 <signal name="5.0V">
@@
 <contactref element="U$1" pad="VBAT"/>
 </signal>
+<signal name="N$4">
+<contactref element="U$1" pad="3"/>
+</signal>
 </signals>

Commit message: PiHat update
Parts:
- added T4: BM08B-SRSS-TB, con-jst2:BM08B-SRSS-TB
- added T4-24-25, T4-30-31, T4-32-33: (no value), SparkFun-Connectors:1X02_NO_SILK
Connections:
- removed net HALL_U0: MOTOR0_SENS.1, U$1.0
- removed net HALL_W0: MOTOR0_SENS.3, U$1.33
- removed net HALL_W1: MOTOR1_SENS.3, U$1.4
- removed net I2C1_SCL: X1.28
- removed net I2C1_SDA: X1.27
- removed net N$4: U$1.3
- removed net SPI_CS1: U$1.31, X1.26
- new net HALL_U0_&_I2C1_SCL: MOTOR0_SENS.1, T4-24-25.2, U$1.29, X1.28
- new net HALL_W0_&_I2C1_SDA: MOTOR0_SENS.3, U$1.30, X1.27
- new net PI_RX: U$1.1, X1.10
- new net PI_TX: U$1.0, X1.8
- new net SPI_CS1_&_HALL_W1: MOTOR1_SENS.3, U$1.14/A0, X1.26
- net HALL_U1: now also T4-32-33.1, U$1.24; no longer U$1.1
- net HALL_V0: now also T4-24-25.1, U$1.32; no longer U$1.24
- net HALL_V1: now also T4-30-31.1, U$1.25; no longer U$1.2
- net I2C0_SCL: now also U$1.19/A5; no longer U$1.29
- net I2C0_SDA: now also U$1.18/A4; no longer U$1.30
- net INH_U0: now also U$1.26, U$1.7
- net INH_V0: now also T4-32-33.2, U$1.33
- net INH_V1: now also U$1.8
- net INH_W0: now also U$1.31
- net INH_W1: now also T4-30-31.2, U$1.28
- net IN_U0: now also T4.1
- net IN_U1: now also T4.6
- net IN_V0: now also T4.2
- net IN_V1: now also T4.7
- net IN_W0: now also T4.4, U$1.10; no longer U$1.21/A7
- net IN_W1: now also T4.8, U$1.9; no longer U$1.10
- net IS_U0: now also U$1.15/A1; no longer U$1.20/A6
- net IS_U1: now also U$1.27; no longer U$1.26
- net IS_V0: now also U$1.20/A6; no longer U$1.19/A5
- net IS_V1: now also U$1.16/A2; no longer U$1.27
- net IS_W0: now also U$1.21/A7; no longer U$1.18/A4
- net IS_W1: now also U$1.17/A3; no longer U$1.28
- net SERVO_0: now also U$1.3; no longer U$1.32
- net SERVO_1: now also U$1.4; no longer U$1.25
- net SPI_CS0: now also U$1.2; no longer U$1.15/A1
- net SPI_SCLK: now also U$1.13; no longer U$1.14/A0
Routing:
- net HALL_U0_&_I2C1_SCL: track 0.00 -> 83.0 mm, vias 0 -> 2
- net SPI_CS1_&_HALL_W1: track 0.00 -> 75.1 mm
- net HALL_W0_&_I2C1_SDA: track 0.00 -> 75.1 mm, vias 0 -> 1
- net IN_W1: track 0.00 -> 71.5 mm
- net IS_V1: track 0.00 -> 68.9 mm
- net SPI_CS0: track 0.00 -> 65.3 mm
- net IN_W0: track 0.00 -> 58.6 mm, vias 0 -> 3
- net PI_TX: track 0.00 -> 51.3 mm, vias 0 -> 3
- net PI_RX: track 0.00 -> 49.7 mm, vias 0 -> 2
- net IN_V0: track 0.00 -> 48.3 mm, vias 0 -> 1
- net IN_U0: track 0.00 -> 47.5 mm
- net GND: track 34.3 -> 80.6 mm
- net HALL_U1: track 0.00 -> 41.2 mm, vias 0 -> 2
- net IN_V1: track 0.00 -> 40.7 mm
- net HALL_V0: track 0.00 -> 40.4 mm
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