File: hardware/EAGLE/projects/PiHatTeensy32/PiHatTeensy32.brd (EAGLE design)
At the start: 100 x 80 mm, 15 parts, among them T4 BM08B-SRSS-TB, U1 TSR_1-2450, X1 RASPI_BOARD_B+_H

Commit message: Befour autorouting
Parts:
- added VCC_RPI: (no value), SparkFun-Connectors:1X02_NO_SILK
- VCC: value JP -> (none)
Connections:
- net SPISCLK renamed SPI_SCLK
- net SPI_CS1_&_HALL_V0 renamed HALL_V0_&_SPI_CS1
- removed net 5V0: X1.2
- new net RPI_5.0V: VCC_RPI.2, X1.2
- net 5.0V: now also VCC_RPI.1
Routing:
- net GND: track 48.7 -> 123.1 mm
- net 5.0V: track 58.0 -> 118.0 mm
- net RPI_5.0V: track 0.00 -> 11.2 mm
- net IN_V1: track 0.74 -> 0.00 mm
- net IN_U1: track 0.59 -> 0.00 mm

Commit message: PiHatMotorController checked
Routing:
- net HALL_U0_&_SPI_MISO: track 0.00 -> 79.4 mm
- net HALL_W0_&_SPI_CS0: track 0.00 -> 75.0 mm
- net IN_W0: track 0.00 -> 70.4 mm, vias 0 -> 2
- net HALL_V0_&_SPI_CS1: track 0.00 -> 65.5 mm, vias 0 -> 1
- net PI_TX: track 0.00 -> 60.9 mm, vias 0 -> 1
- net PI_RX: track 0.00 -> 53.7 mm
- net IS_U0: track 0.00 -> 49.1 mm
- net IN_U0: track 0.00 -> 47.4 mm
- net IN_W1: track 0.00 -> 47.2 mm, vias 0 -> 1
- net IN_V1: track 0.00 -> 45.8 mm, vias 0 -> 3
- net IN_V0: track 0.51 -> 46.3 mm, vias 0 -> 1
- net IS_V1: track 0.00 -> 43.4 mm, vias 0 -> 1
- net SERVO_1: track 0.05 -> 43.2 mm
- net HALL_W1: track 0.00 -> 42.9 mm
- net SERVO_0: track 0.00 -> 42.4 mm
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
Commit message: wired HALL_V1 to Pin 7
Connections:
- removed net TBA5: U$1.7
- net HALL_V1: now also U$1.7
Routing:
- net HALL_V1: track 0.00 -> 28.0 mm, vias 0 -> 2
Changed lines of the file:
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@@
 <?xml version="1.0" encoding="utf-8"?>
 <!DOCTYPE eagle SYSTEM "eagle.dtd">
-<eagle version="9.6.0">
+<eagle version="9.5.2">
 <drawing>
 <settings>
@@
 <wire x1="33.655" y1="50.165" x2="30.1625" y2="50.165" width="0.3048" layer="1"/>
 </signal>
-<signal name="TBA5">
-<contactref element="U$1" pad="7"/>
-</signal>
 <signal name="HALL_V1">
 <contactref element="MOTOR1_SENS" pad="2"/>
+<contactref element="U$1" pad="7"/>
+<wire x1="57.15" y1="13.97" x2="46.355" y2="24.765" width="0.3048" layer="1"/>
+<via x="46.355" y="24.765" extent="1-16" drill="0.35"/>
+<wire x1="46.355" y1="24.765" x2="46.355" y2="31.75" width="0.3048" layer="16"/>
+<via x="46.355" y="31.75" extent="1-16" drill="0.35"/>
+<wire x1="46.355" y1="31.75" x2="40.64" y2="31.75" width="0.3048" layer="1"/>
 </signal>
 <signal name="SPI_MOSI">
