File: hardware/EAGLE/projects/PiHatTeensy32/PiHatTeensy32.sch (EAGLE design)
At the start: 15 parts, among them T4 BM08B-SRSS-TB, U1 TSR_1-2450, X1 RASPI_BOARD_B+_H

Commit message: Befour autorouting
Parts:
- added VCC_RPI: (no value), SparkFun-Connectors:CONN_021X02_NO_SILK
- VCC: value JP -> (none)
Connections:
- net SPISCLK renamed SPI_SCLK
- net SPI_CS1_&_HALL_V0 renamed HALL_V0_&_SPI_CS1
- new net RPI_5.0V: VCC_RPI.2, X1.5V0
- net 5.0V: now also VCC_RPI.1
Other:
- moved on the sheet: BATTERY, C0, MOTOR0_CONTROL, MOTOR0_SENS, MOTOR1_CONTROL, MOTOR1_SENS, T4-1, T4-2, T4-24-25, T4-3, T4-30-31, T4-32-33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

Commit message: wired HALL_V1 to Pin 7
Connections:
- removed net TBA5: U$1.7/RX3
- net HALL_V1: now also U$1.7/RX3
Changed lines of the file:
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@@
 <?xml version="1.0" encoding="utf-8"?>
 <!DOCTYPE eagle SYSTEM "eagle.dtd">
-<eagle version="9.6.0">
+<eagle version="9.5.2">
 <drawing>
 <settings>
@@
 </segment>
 </net>
-<net name="TBA5" class="0">
+<net name="HALL_V1" class="0">
+<segment>
+<wire x1="10.16" y1="-60.96" x2="20.32" y2="-60.96" width="0.1524" layer="91"/>
+<label x="20.32" y="-60.96" size="1.778" layer="95" xref="yes"/>
+<pinref part="MOTOR1_SENS" gate="G$1" pin="2"/>
+</segment>
 <segment>
 <pinref part="U$1" gate="G$1" pin="7/RX3"/>
@@
 </segment>
 </net>
-<net name="HALL_V1" class="0">
-<segment>
-<wire x1="10.16" y1="-60.96" x2="20.32" y2="-60.96" width="0.1524" layer="91"/>
-<label x="20.32" y="-60.96" size="1.778" layer="95" xref="yes"/>
-<pinref part="MOTOR1_SENS" gate="G$1" pin="2"/>
-</segment>
-</net>

Commit message: cancelled UART, made some cosmetic changes, ready for production
Connections:
- net HALL_U1: now also U$1.0/RX1/T; no longer T4-32-33.1, U$1.24
- net HALL_V1: now also U$1.1/TX1/T; no longer U$1.7/RX3
- net HALL_W1: now also U$1.7/RX3; no longer U$1.32/T/PWM
- net PI_RX: no longer U$1.1/TX1/T
- net PI_TX: no longer U$1.0/RX1/T
Changed lines of the file:
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@@
 </segment>
 <segment>
-<pinref part="U$1" gate="G$1" pin="24"/>
-<wire x1="165.1" y1="-124.46" x2="157.48" y2="-124.46" width="0.1524" layer="91"/>
-<label x="157.48" y="-124.46" size="1.778" layer="95" rot="R180" xref="yes"/>
-</segment>
-<segment>
-<pinref part="T4-32-33" gate="G$1" pin="1"/>
-<wire x1="10.16" y1="-76.2" x2="53.34" y2="-76.2" width="0.1524" layer="91"/>
-<label x="53.34" y="-76.2" size="1.778" layer="95" xref="yes"/>
+<pinref part="U$1" gate="G$1" pin="0/RX1/T"/>
+<wire x1="165.1" y1="-63.5" x2="157.48" y2="-63.5" width="0.1524" layer="91"/>
+<label x="157.48" y="-63.5" size="1.778" layer="95" rot="R180" xref="yes"/>
 </segment>
 </net>
@@
 <label x="220.98" y="-30.48" size="1.778" layer="95" xref="yes"/>
 </segment>
-<segment>
-<pinref part="U$1" gate="G$1" pin="0/RX1/T"/>
-<wire x1="165.1" y1="-63.5" x2="157.48" y2="-63.5" width="0.1524" layer="91"/>
-<label x="157.48" y="-63.5" size="1.778" layer="95" rot="R180" xref="yes"/>
-</segment>
 </net>
 <net name="PI_RX" class="0">
@@
 <wire x1="200.66" y1="-33.02" x2="205.74" y2="-33.02" width="0.1524" layer="91"/>
 <label x="205.74" y="-33.02" size="1.778" layer="95" xref="yes"/>
-</segment>
-<segment>
-<pinref part="U$1" gate="G$1" pin="1/TX1/T"/>
-<wire x1="165.1" y1="-66.04" x2="124.46" y2="-66.04" width="0.1524" layer="91"/>
-<label x="124.46" y="-66.04" size="1.778" layer="95" rot="R180" xref="yes"/>
 </segment>
 </net>
@@
 </segment>
 <segment>
-<pinref part="U$1" gate="G$1" pin="7/RX3"/>
-<wire x1="165.1" y1="-81.28" x2="124.46" y2="-81.28" width="0.1524" layer="91"/>
-<label x="124.46" y="-81.28" size="1.778" layer="95" rot="R180" xref="yes"/>
+<pinref part="U$1" gate="G$1" pin="1/TX1/T"/>
+<wire x1="165.1" y1="-66.04" x2="124.46" y2="-66.04" width="0.1524" layer="91"/>
+<label x="124.46" y="-66.04" size="1.778" layer="95" rot="R180" xref="yes"/>
 </segment>
 </net>
@@
 </segment>
 <segment>
-<pinref part="U$1" gate="G$1" pin="32/T/PWM"/>
-<wire x1="210.82" y1="-106.68" x2="248.92" y2="-106.68" width="0.1524" layer="91"/>
-<label x="248.92" y="-106.68" size="1.778" layer="95" xref="yes"/>
+<pinref part="U$1" gate="G$1" pin="7/RX3"/>
+<wire x1="165.1" y1="-81.28" x2="124.46" y2="-81.28" width="0.1524" layer="91"/>
+<label x="124.46" y="-81.28" size="1.778" layer="95" rot="R180" xref="yes"/>
 </segment>
 </net>

Commit message: uart tx tx added back again, more coesmetic changes
Connections:
- removed net HALL_U1: MOTOR1_SENS.1, U$1.0/RX1/T
- removed net HALL_V1: MOTOR1_SENS.2, U$1.1/TX1/T
- removed net PI_RX: X1.RXD
- removed net PI_TX: X1.TXD
- new net HALL_U1_&_PI_TX: MOTOR1_SENS.1, U$1.0/RX1/T, X1.TXD
- new net HALL_V1_&PI_RX: MOTOR1_SENS.2, U$1.1/TX1/T, X1.RXD
Changed lines of the file:
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@@
-</segment>
-</net>
-<net name="HALL_U1" class="0">
-<segment>
-<wire x1="10.16" y1="-63.5" x2="53.34" y2="-63.5" width="0.1524" layer="91"/>
-<label x="53.34" y="-63.5" size="1.778" layer="95" xref="yes"/>
-<pinref part="MOTOR1_SENS" gate="G$1" pin="1"/>
-</segment>
-<segment>
-<pinref part="U$1" gate="G$1" pin="0/RX1/T"/>
-<wire x1="165.1" y1="-63.5" x2="157.48" y2="-63.5" width="0.1524" layer="91"/>
-<label x="157.48" y="-63.5" size="1.778" layer="95" rot="R180" xref="yes"/>
 </segment>
 </net>
@@
 </segment>
 </net>
-<net name="PI_TX" class="0">
-<segment>
-<pinref part="X1" gate="G$1" pin="TXD"/>
-<wire x1="200.66" y1="-30.48" x2="220.98" y2="-30.48" width="0.1524" layer="91"/>
-<label x="220.98" y="-30.48" size="1.778" layer="95" xref="yes"/>
-</segment>
-</net>
-<net name="PI_RX" class="0">
-<segment>
-<pinref part="X1" gate="G$1" pin="RXD"/>
-<wire x1="200.66" y1="-33.02" x2="205.74" y2="-33.02" width="0.1524" layer="91"/>
-<label x="205.74" y="-33.02" size="1.778" layer="95" xref="yes"/>
-</segment>
-</net>
 <net name="I2C1_SDA" class="0">
 <segment>
@@
 <wire x1="200.66" y1="7.62" x2="236.22" y2="7.62" width="0.1524" layer="91"/>
 <label x="236.22" y="7.62" size="1.778" layer="95" xref="yes"/>
-</segment>
-</net>
-<net name="HALL_V1" class="0">
-<segment>
-<wire x1="10.16" y1="-60.96" x2="20.32" y2="-60.96" width="0.1524" layer="91"/>
-<label x="20.32" y="-60.96" size="1.778" layer="95" xref="yes"/>
-<pinref part="MOTOR1_SENS" gate="G$1" pin="2"/>
-</segment>
-<segment>
-<pinref part="U$1" gate="G$1" pin="1/TX1/T"/>
-<wire x1="165.1" y1="-66.04" x2="124.46" y2="-66.04" width="0.1524" layer="91"/>
-<label x="124.46" y="-66.04" size="1.778" layer="95" rot="R180" xref="yes"/>
 </segment>
 </net>
@@
 </segment>
 </net>
+<net name="HALL_U1_&amp;_PI_TX" class="0">
+<segment>
+<pinref part="U$1" gate="G$1" pin="0/RX1/T"/>
+<wire x1="165.1" y1="-63.5" x2="157.48" y2="-63.5" width="0.1524" layer="91"/>
+<label x="157.48" y="-63.5" size="1.778" layer="95" rot="R180" xref="yes"/>
+</segment>
+<segment>
+<pinref part="X1" gate="G$1" pin="TXD"/>
+<wire x1="200.66" y1="-30.48" x2="220.98" y2="-30.48" width="0.1524" layer="91"/>
+<label x="220.98" y="-30.48" size="1.778" layer="95" xref="yes"/>
+</segment>
+<segment>
+<wire x1="10.16" y1="-63.5" x2="53.34" y2="-63.5" width="0.1524" layer="91"/>
+<label x="53.34" y="-63.5" size="1.778" layer="95" xref="yes"/>
+<pinref part="MOTOR1_SENS" gate="G$1" pin="1"/>
+</segment>
+</net>
+<net name="HALL_V1_&amp;PI_RX" class="0">
+<segment>
+<pinref part="U$1" gate="G$1" pin="1/TX1/T"/>
+<wire x1="165.1" y1="-66.04" x2="124.46" y2="-66.04" width="0.1524" layer="91"/>
+<label x="124.46" y="-66.04" size="1.778" layer="95" rot="R180" xref="yes"/>
+</segment>
+<segment>
+<pinref part="X1" gate="G$1" pin="RXD"/>
+<wire x1="200.66" y1="-33.02" x2="205.74" y2="-33.02" width="0.1524" layer="91"/>
+<label x="205.74" y="-33.02" size="1.778" layer="95" xref="yes"/>
+</segment>
+<segment>
+<wire x1="10.16" y1="-60.96" x2="20.32" y2="-60.96" width="0.1524" layer="91"/>
+<label x="20.32" y="-60.96" size="1.778" layer="95" xref="yes"/>
+<pinref part="MOTOR1_SENS" gate="G$1" pin="2"/>
+</segment>
+</net>

Commit message: Label added to PiHatTeensy32
Parts:
- renumbered U$1 to TEENSY, U1 to DC-DC
