File: hardware/EAGLE/projects/PiHatTeensy32_40/PiHatTeensy32_40.brd (EAGLE design)
At the start: 100 x 80 mm, 15 parts, among them T4 BM08B-SRSS-TB, U1 TSR_1-2450, X1 RASPI_BOARD_B+_H

Commit message: latest changes
Parts:
- removed T4: BM08B-SRSS-TB, con-jst2:BM08B-SRSS-TB
- removed T4-24-25, T4-30-31, T4-32-33: (no value), SparkFun-Connectors:1X02_NO_SILK
Connections:
- removed net HALL_U0_&_SPI_MISO: MOTOR0_SENS.1, U$1.12, X1.21
- removed net HALL_W0_&_SPI_CS0: MOTOR0_SENS.3, U$1.2, X1.24
- removed net PI_RX: U$1.1, X1.10
- removed net PI_TX: U$1.0, X1.8
- removed net SPISCLK: U$1.13, X1.23
- removed net SPI_CS1_&_HALL_V0: MOTOR0_SENS.2, U$1.14/A0, X1.26
- removed net TBA5: U$1.7
- new net HALL_U0: MOTOR0_SENS.1, U$1.0
- new net HALL_V0: MOTOR0_SENS.2, U$1.24
- new net HALL_W0: MOTOR0_SENS.3, U$1.33
- new net N$4: U$1.3
- new net SPI_CS0: U$1.15/A1, X1.24
- new net SPI_CS1: U$1.31, X1.26
- new net SPI_MISO: U$1.12, X1.21
- new net SPI_SCLK: U$1.14/A0, X1.23
- net HALL_U1: now also U$1.1; no longer T4-32-33.1, U$1.24
- net HALL_V1: now also U$1.2
- net HALL_W1: now also U$1.4; no longer U$1.32
- net I2C0_SCL: now also U$1.29; no longer U$1.19/A5
- net I2C0_SDA: now also U$1.30; no longer U$1.18/A4
- net I2C1_SCL: no longer T4-24-25.2, U$1.29
- net I2C1_SDA: no longer T4-24-25.1, U$1.30
- net INH_U0: no longer U$1.26
- net INH_U1: no longer T4-30-31.1, U$1.25
- net INH_V0: no longer T4-32-33.2, U$1.33
- net INH_V1: no longer U$1.8
- net INH_W0: no longer U$1.31
- net INH_W1: no longer T4-30-31.2, U$1.28
- net IN_U0: no longer T4.1
- net IN_U1: no longer T4.6
- net IN_V0: no longer T4.2
- net IN_V1: no longer T4.7
- net IN_W0: now also U$1.21/A7; no longer T4.4, U$1.10
- net IN_W1: now also U$1.10; no longer T4.8, U$1.9
- net IS_U0: now also U$1.20/A6; no longer U$1.15/A1
- net IS_U1: now also U$1.26; no longer U$1.27
- net IS_V0: now also U$1.19/A5; no longer U$1.20/A6
- net IS_V1: now also U$1.27; no longer U$1.16/A2
- net IS_W0: now also U$1.18/A4; no longer U$1.21/A7
- net IS_W1: now also U$1.28; no longer U$1.17/A3
- net SERVO_0: now also U$1.32; no longer U$1.3
- net SERVO_1: now also U$1.25; no longer U$1.4
Routing:
- net GND: track 48.7 -> 34.3 mm
- net IN_V1: track 0.74 -> 0.00 mm
- net IN_U1: track 0.59 -> 0.00 mm
- net IN_V0: track 0.51 -> 0.00 mm
