File: hardware/EAGLE/projects/PiHatTeensy32_40/PiHatTeensy32_40.sch (EAGLE design)
At the start: 15 parts, among them T4 BM08B-SRSS-TB, U1 TSR_1-2450, X1 RASPI_BOARD_B+_H

Commit message: latest changes
Parts:
- removed T4: BM08B-SRSS-TB, con-jst2:BM08B-SRSS-TB
- removed T4-24-25, T4-30-31, T4-32-33: (no value), SparkFun-Connectors:CONN_021X02_NO_SILK
Connections:
- removed net HALL_U0_&_SPI_MISO: MOTOR0_SENS.1, U$1.12/MISO, X1.SPI_MISO
- removed net HALL_W0_&_SPI_CS0: MOTOR0_SENS.3, U$1.2, X1.SPI_CE0
- removed net PI_RX: U$1.1/TX1/T, X1.RXD
- removed net PI_TX: U$1.0/RX1/T, X1.TXD
- removed net SPISCLK: U$1.13/SCK/LED, X1.SPI_SCLK
- removed net SPI_CS1_&_HALL_V0: MOTOR0_SENS.2, U$1.14/A0, X1.SPI_CE1
- removed net TBA5: U$1.7/RX3
- new net HALL_U0: MOTOR0_SENS.1, U$1.0/RX1/T
- new net HALL_V0: MOTOR0_SENS.2, U$1.24
- new net HALL_W0: MOTOR0_SENS.3, U$1.33/T
- new net N$4: U$1.3/CAN-TX/PWM
- new net SPI_CS0: U$1.15/A1/T, X1.SPI_CE0
- new net SPI_CS1: U$1.31/A20, X1.SPI_CE1
- new net SPI_MISO: U$1.12/MISO, X1.SPI_MISO
- new net SPI_SCLK: U$1.14/A0, X1.SPI_SCLK
- net HALL_U1: now also U$1.1/TX1/T; no longer T4-32-33.1, U$1.24
- net HALL_V1: now also U$1.2
- net HALL_W1: now also U$1.4/CAN-RX/PWM; no longer U$1.32/T/PWM
- net I2C0_SCL: now also U$1.29/A18/SCL1; no longer U$1.19/A5/T/SCL0
- net I2C0_SDA: now also U$1.30/A19/SDA1; no longer U$1.18/A4/T/SDA0
- net I2C1_SCL: no longer T4-24-25.2, U$1.29/A18/SCL1
- net I2C1_SDA: no longer T4-24-25.1, U$1.30/A19/SDA1
- net INH_U0: no longer U$1.26/A15
- net INH_U1: no longer T4-30-31.1, U$1.25/T/PWM
- net INH_V0: no longer T4-32-33.2, U$1.33/T
- net INH_V1: no longer U$1.8/TX3
- net INH_W0: no longer U$1.31/A20
- net INH_W1: no longer T4-30-31.2, U$1.28/A17
- net IN_U0: no longer T4-1.S
- net IN_U1: no longer T4-6.S
- net IN_V0: no longer T4-2.S
- net IN_V1: no longer T4-7.S
- net IN_W0: now also U$1.21/A7/PWM; no longer T4-4.S, U$1.10/TX2/PWM
- net IN_W1: now also U$1.10/TX2/PWM; no longer T4-8.S, U$1.9/RX2/PWM
- net IS_U0: now also U$1.20/A6/PWM; no longer U$1.15/A1/T
- net IS_U1: now also U$1.26/A15; no longer U$1.27/A16
- net IS_V0: now also U$1.19/A5/T/SCL0; no longer U$1.20/A6/PWM
- net IS_V1: now also U$1.27/A16; no longer U$1.16/A2/T
- net IS_W0: now also U$1.18/A4/T/SDA0; no longer U$1.21/A7/PWM
- net IS_W1: now also U$1.28/A17; no longer U$1.17/A3/T
- net SERVO_0: now also U$1.32/T/PWM; no longer U$1.3/CAN-TX/PWM
- net SERVO_1: now also U$1.25/T/PWM; no longer U$1.4/CAN-RX/PWM
